File: hw/calaos_plc_io/calaos_plc_io_outputs-1.sch (KiCad schematic (older format))
At the start: 9 parts, among them Q1 Q_NPN_BCE, U3 LTV-847, U9 PCA9505

Commit message: More values for resistances and capa
Parts:
- Q1: Estimated price (none) -> 0.1; Mouser Ref (none) -> 863-MMBT2222ALT1G
- R10: footprint (none) -> Resistors_SMD:R_0603
- R11, R12: value 10k -> 4k7; footprint (none) -> Resistors_SMD:R_0603
- R13, R9: footprint Resistors_SMD:R_0805 -> Resistors_SMD:R_0603
- U9: footprint (none) -> Housings_SSOP:TSSOP-56_6.1x14mm_Pitch0.5mm
- U9: footprint (none) -> Housings_SSOP:TSSOP-56_6.1x14mm_Pitch0.5mm; Estimated Price (none) -> 3.74; Mouser Ref (none) -> 771-PCA9505DGG-T
Connections:
- wire segments 40 -> 42
Changed lines of the file:
@@
 LIBS:74xgxx
 LIBS:pca9505
+LIBS:calaos_plc_io-cache
 EELAYER 25 0
 EELAYER END
@@
 	2400 2900 2800 2900
 $Comp
-L GNDREF #PWR39
+L GNDREF #PWR041
 U 1 1 55D96BF9
 P 4350 3250
-F 0 "#PWR39" H 4350 3000 50  0001 C CNN
+F 0 "#PWR041" H 4350 3000 50  0001 C CNN
 F 1 "GNDREF" H 4350 3100 50  0000 C CNN
 F 2 "" H 4350 3250 60  0000 C CNN
@@
 F 1 "Q_NPN_BCE" H 4850 2850 50  0000 R CNN
 F 2 "SMD_Packages:POT_SMD" H 4450 3000 29  0001 C CNN
-F 3 "" H 4250 2900 60  0000 C CNN
+F 3 "http://www.mouser.com/ds/2/308/MMBT2222LT1-D-80103.pdf" H 4250 2900 60  0001 C CNN
+F 4 "863-MMBT2222ALT1G " H 4250 2900 60  0001 C CNN "Mouser Ref"
+F 5 "0.1" H 4250 2900 60  0001 C CNN "Estimated price"
 	1    4250 2900
 	1    0    0    -1
@@
 F 0 "R9" V 4030 2400 50  0000 C CNN
 F 1 "10k" V 3950 2400 50  0000 C CNN
-F 2 "Resistors_SMD:R_0805" V 3880 2400 30  0001 C CNN
+F 2 "Resistors_SMD:R_0603" V 3880 2400 30  0001 C CNN
 F 3 "" H 3950 2400 30  0000 C CNN
 	1    3950 2400
@@
 F 0 "R13" V 4430 2400 50  0000 C CNN
 F 1 "10k" V 4350 2400 50  0000 C CNN
-F 2 "Resistors_SMD:R_0805" V 4280 2400 30  0001 C CNN
+F 2 "Resistors_SMD:R_0603" V 4280 2400 30  0001 C CNN
 F 3 "" H 4350 2400 30  0000 C CNN
 	1    4350 2400
@@
 $EndComp
 $Comp
-L +24V #PWR38
+L +24V #PWR042
 U 1 1 55D96BF2
 P 4150 2100
-F 0 "#PWR38" H 4150 1950 50  0001 C CNN
+F 0 "#PWR042" H 4150 1950 50  0001 C CNN
 F 1 "+24V" H 4150 2240 50  0000 C CNN
 F 2 "" H 4150 2100 60  0000 C CNN
@@
 F 0 "D3" H 2950 3200 50  0000 C CNN
 F 1 "LED" H 2950 3000 50  0000 C CNN
-F 2 "" H 2950 3100 60  0000 C CNN
+F 2 "" H 2950 3100 60  0001 C CNN
 F 3 "" H 2950 3100 60  0000 C CNN
 	1    2950 3100
@@
 F 0 "R10" V 2850 2900 50  0000 C CNN
 F 1 "220" V 2950 2900 50  0000 C CNN
-F 2 "" V 2880 2900 30  0000 C CNN
+F 2 "Resistors_SMD:R_0603" V 2880 2900 30  0001 C CNN
 F 3 "" H 2950 2900 30  0000 C CNN
 	1    2950 2900
@@
 	3250 3100 3150 3100
 $Comp
-L GND #PWR37
+L GND #PWR043
 U 1 1 55DF000A
 P 2650 3200
-F 0 "#PWR37" H 2650 2950 50  0001 C CNN
+F 0 "#PWR043" H 2650 2950 50  0001 C CNN
 F 1 "GND" H 2650 3050 50  0000 C CNN
 F 2 "" H 2650 3200 60  0000 C CNN
@@
 F 0 "U9" H 2150 9400 60  0000 C CNN
 F 1 "PCA9505" H 2250 8150 60  0000 C CNN
-F 2 "" H 2250 8150 60  0000 C CNN
+F 2 "Housings_SSOP:TSSOP-56_6.1x14mm_Pitch0.5mm" H 2250 8150 60  0001 C CNN
 F 3 "" H 2250 8150 60  0000 C CNN
 	1    2050 8800
@@
 F 0 "U9" H 3650 9350 60  0000 C CNN
 F 1 "PCA9505" H 3750 8100 60  0000 C CNN
-F 2 "" H 3750 8100 60  0000 C CNN
+F 2 "Housings_SSOP:TSSOP-56_6.1x14mm_Pitch0.5mm" H 3750 8100 60  0001 C CNN
 F 3 "" H 3750 8100 60  0000 C CNN
 	2    3550 8750
@@
 F 0 "U9" H 5100 9400 60  0000 C CNN
 F 1 "PCA9505" H 5200 8150 60  0000 C CNN
-F 2 "" H 5200 8150 60  0000 C CNN
+F 2 "Housings_SSOP:TSSOP-56_6.1x14mm_Pitch0.5mm" H 5200 8150 60  0001 C CNN
 F 3 "" H 5200 8150 60  0000 C CNN
 	3    5000 8800
@@
 F 0 "U9" H 6400 9300 60  0000 C CNN
 F 1 "PCA9505" H 6500 8050 60  0000 C CNN
-F 2 "" H 6500 8050 60  0000 C CNN
+F 2 "Housings_SSOP:TSSOP-56_6.1x14mm_Pitch0.5mm" H 6500 8050 60  0001 C CNN
 F 3 "" H 6500 8050 60  0000 C CNN
 	4    6300 8700
@@
 F 0 "U9" H 7650 9350 60  0000 C CNN
 F 1 "PCA9505" H 7750 8100 60  0000 C CNN
-F 2 "" H 7750 8100 60  0000 C CNN
+F 2 "Housings_SSOP:TSSOP-56_6.1x14mm_Pitch0.5mm" H 7750 8100 60  0001 C CNN
 F 3 "" H 7750 8100 60  0000 C CNN
 	5    7550 8750
@@
 F 0 "U9" H 13200 2750 60  0000 C CNN
 F 1 "PCA9505" H 13200 2000 60  0000 C CNN
-F 2 "" H 13300 1500 60  0000 C CNN
-F 3 "" H 13300 1500 60  0000 C CNN
+F 2 "Housings_SSOP:TSSOP-56_6.1x14mm_Pitch0.5mm" H 13300 1500 60  0001 C CNN
+F 3 "http://www.mouser.com/ds/2/302/PCA9505_9506-352364.pdf" H 13300 1500 60  0001 C CNN
+F 4 "771-PCA9505DGG-T" H 13100 2150 60  0001 C CNN "Mouser Ref"
+F 5 "3.74" H 13100 2150 60  0001 C CNN "Estimated Price"
 	6    13100 2150
 	1    0    0    -1
@@
 F 0 "U9" V 13550 3750 60  0000 C CNN
 F 1 "PCA9505" V 12750 3850 60  0000 C CNN
-F 2 "" H 13350 3050 60  0000 C CNN
+F 2 "Housings_SSOP:TSSOP-56_6.1x14mm_Pitch0.5mm" H 13350 3050 60  0001 C CNN
 F 3 "" H 13350 3050 60  0000 C CNN
 	7    13150 3700
@@
 $EndComp
 $Comp
-L +5V #PWR42
+L +5V #PWR044
 U 1 1 55E1AEA9
 P 13150 2950
-F 0 "#PWR42" H 13150 2800 50  0001 C CNN
+F 0 "#PWR044" H 13150 2800 50  0001 C CNN
 F 1 "+5V" H 13150 3090 50  0000 C CNN
 F 2 "" H 13150 2950 60  0000 C CNN
@@
 Connection ~ 13150 3050
 $Comp
-L GND #PWR43
+L GND #PWR045
 U 1 1 55E1AF46
 P 13150 4150
-F 0 "#PWR43" H 13150 3900 50  0001 C CNN
+F 0 "#PWR045" H 13150 3900 50  0001 C CNN
 F 1 "GND" H 13150 4000 50  0000 C CNN
 F 2 "" H 13150 4150 60  0000 C CNN
@@
 P 12050 1750
 F 0 "R11" V 12130 1750 50  0000 C CNN
-F 1 "10k" V 12050 1750 50  0000 C CNN
-F 2 "" V 11980 1750 30  0000 C CNN
+F 1 "4k7" V 12050 1750 50  0000 C CNN
+F 2 "Resistors_SMD:R_0603" V 11980 1750 30  0001 C CNN
 F 3 "" H 12050 1750 30  0000 C CNN
 	1    12050 1750
@@
 	12050 1950 12050 1900
 $Comp
-L GND #PWR41
+L GND #PWR046
 U 1 1 55E1B52C
 P 12400 2300
-F 0 "#PWR41" H 12400 2050 50  0001 C CNN
+F 0 "#PWR046" H 12400 2050 50  0001 C CNN
 F 1 "GND" H 12400 2150 50  0000 C CNN
 F 2 "" H 12400 2300 60  0000 C CNN
@@
 $EndComp
 $Comp
-L +5V #PWR40
+L +5V #PWR047
 U 1 1 55E1B5E1
 P 12050 1500
-F 0 "#PWR40" H 12050 1350 50  0001 C CNN
+F 0 "#PWR047" H 12050 1350 50  0001 C CNN
 F 1 "+5V" H 12050 1640 50  0000 C CNN
 F 2 "" H 12050 1500 60  0000 C CNN
@@
 P 13700 1550
 F 0 "R12" V 13780 1550 50  0000 C CNN
-F 1 "10k" V 13700 1550 50  0000 C CNN
-F 2 "" V 13630 1550 30  0000 C CNN
+F 1 "4k7" V 13700 1550 50  0000 C CNN
+F 2 "Resistors_SMD:R_0603" V 13630 1550 30  0001 C CNN
 F 3 "" H 13700 1550 30  0000 C CNN
 	1    13700 1550
@@
 $EndComp
 $Comp
-L +5V #PWR44
+L +5V #PWR048
 U 1 1 55E1DCFF
 P 13700 1300
-F 0 "#PWR44" H 13700 1150 50  0001 C CNN
+F 0 "#PWR048" H 13700 1150 50  0001 C CNN
 F 1 "+5V" H 13700 1440 50  0000 C CNN
 F 2 "" H 13700 1300 60  0000 C CNN
@@
 Wire Wire Line
 	13600 1900 13700 1900
+$Comp
+L GND #PWR049
+U 1 1 55DAE293
+P 13700 2100
+F 0 "#PWR049" H 13700 1850 50  0001 C CNN
+F 1 "GND" H 13700 1950 50  0000 C CNN
+F 2 "" H 13700 2100 60  0000 C CNN
+F 3 "" H 13700 2100 60  0000 C CNN
+	1    13700 2100
+	1    0    0    -1
+$EndComp
+Wire Wire Line
+	13600 2000 13700 2000
+Wire Wire Line
+	13700 2000 13700 2100
 $EndSCHEMATC
