File: hw/calaos_plc_io/calaos_plc_io.sch (KiCad schematic (older format))
At the start: 32 parts, among them J1 RJ12, P1 CONN_01X03, P2 CONN_01X06, P3 CONN_01X40, P4 CONN_01X40, U1 LM7824CT, U2 LM7805CT, U4 LD1117S33TR, U5 MAX485, U6 STM32F030K6, Y1 Crystal

Commit message: More values for resistances and capa
Parts:
- C1: value C -> 0.33uF; footprint (none) -> Capacitors_SMD:C_0603
- C10, C11, C12, C13, C14, C9: value C -> 100nF; footprint (none) -> Capacitors_SMD:C_0603
- C2, C4, C7, C8: footprint (none) -> Capacitors_SMD:C_0603
- C3: value C -> 0.1uF; footprint (none) -> Capacitors_SMD:C_0603
- C5, C6: value C -> 20pF; footprint (none) -> Capacitors_SMD:C_0603
- P3, P4: footprint (none) -> Pin_Headers:Pin_Header_Straight_1x40
- R1: value R -> 120; footprint (none) -> Resistors_SMD:R_0603
- R2: value R -> 10k; footprint (none) -> Resistors_SMD:R_0603
- R3: value R -> 510; footprint (none) -> Resistors_SMD:R_0603
- R4: value 120 -> 510; footprint (none) -> Resistors_SMD:R_0603
- U1: footprint TO-220 -> Power_Integrations:TO-220; Estimated price (none) -> 0.64; Mouser Ref (none) -> 512-LM7824CT
- U2: footprint TO-220 -> Power_Integrations:TO-220; Estimated price (none) -> 0.631; Mouser Ref (none) -> 512-LM7805CT
- U4: footprint SOT-223 -> TO_SOT_Packages_SMD:SOT-223; Estimated price (none) -> 0.959; Mouser Ref (none) -> 926-LM1117MPX3.3NOPB
- U5: footprint (none) -> Housings_SOIC:SOIC-8_3.9x4.9mm_Pitch1.27mm; Estimated price (none) -> 1.34; Mouser Ref (none) -> 968-ISL83490IBZ
- U6: footprint LQFP-32 -> Housings_QFP:TQFP-32_7x7mm_Pitch0.8mm; Estimated price (none) -> 1.4; Mouser Ref (none) -> 511-STM32F030K6T6
- Y1: value Crystal -> 8MHz; footprint (none) -> Crystals:Crystal_HC48-U_Vertical
- gave numbers to parts that had none: 1
Connections:
- wire segments 147 -> 137
- no-connect marks 1 -> 15

Commit message: Update schematics
Parts:
- removed P3, P4: CONN_01X40, Pin_Headers:Pin_Header_Straight_1x40, symbol CONN_01X40
- added P3, P4: CONN_01X20, Pin_Headers:Pin_Header_Straight_1x20, symbol CONN_01X20
- D100: renamed from D1; footprint (none) -> LEDs:LED-0603
- JP1: footprint (none) -> Pin_Headers:Pin_Header_Straight_1x02
- P1: footprint (none) -> Pin_Headers:Pin_Header_Straight_1x03
- P2: footprint (none) -> Pin_Headers:Pin_Header_Straight_1x06
- P5: footprint (none) -> Pin_Headers:Pin_Header_Straight_1x04
- Y1: footprint Crystals:Crystal_HC48-U_Vertical -> Crystals_Oscillators_SMD:crystal_FA238-TSX3225
Connections:
- net labels added: INT
- net labels removed: INT_INPUTS, INT_OUTPUTS
- wire segments 137 -> 171
- no-connect marks 15 -> 16

Commit message: Add pcb with placement of components
Parts:
- removed J1: RJ12, symbol RJ12
- removed JP1: JUMPER, Pin_Headers:Pin_Header_Straight_1x02, symbol JUMPER
- removed P1: CONN_01X03, Pin_Headers:Pin_Header_Straight_1x03, symbol CONN_01X03
- removed P3, P4: CONN_01X20, Pin_Headers:Pin_Header_Straight_1x20, symbol CONN_01X20
- removed R2: 10k, Resistors_SMD:R_0603, symbol R
- removed R3: 510, Resistors_SMD:R_0603, symbol R
- removed U5: MAX485, Housings_SOIC:SOIC-8_3.9x4.9mm_Pitch1.27mm, symbol MAX485
- removed U6: STM32F030K6, Housings_QFP:TQFP-32_7x7mm_Pitch0.8mm, symbol STM32F030K6
- added C15: 100nF, Capacitors_SMD:C_0603, symbol C
- added CON1, CON2: TerminalBlock, plc:Terminalblock_1708084, symbol TerminalBlock
- added JP1: Jumper_NO_Small, Wire_Pads:SolderWirePad_2x_0-8mmDrill, symbol Jumper_NO_Small
- added P4: CONN_01X04, plc:Terminalbloc_1726040, symbol CONN_01X04
- added R99: 120, Resistors_SMD:R_0603, symbol R
- added U4: STM32F105R8, Housings_QFP:LQFP-64_10x10mm_Pitch0.5mm, symbol STM32F105R8
- added U5: MCP2551-I/SN, Housings_SOIC:SOIC-8_3.9x4.9mm_Pitch1.27mm, symbol MCP2551-I/SN
- R1: value 120 -> 1k
- renumbered C5 to C1, C8 to C10, C6 to C2, C1 to C3, C2 to C4, C3 to C5, C4 to C6, C9 to C8, C10 to C9, D100 to D1, P5 to P1, R4 to R2, U4 to U3
Connections:
- net labels added: +3.3V, CANH, CANL, CAN_RX, CAN_TX, O_0, O_1, O_10, O_11, O_12, O_13, O_14, O_15, O_2, O_3, O_4, O_5, O_6, O_7, O_8, O_9, RS485_CTS, RS485_RX, RS485_TX
- net labels removed: A, B, CTS, INT, RX, SCA, SCL, TX
- wire segments 171 -> 197
- no-connect marks 16 -> 1
Other:
- note removed: "Analaog value used to fix an hardware revision"
- note removed: "Terminal\nresistor"
- moved on the sheet: C1, C10, C11, C12, C13, C14, C2, C3, C4, C5, C6, C7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

Commit message: Update schematics and pcb
Parts:
- removed U1: LM7824CT, Power_Integrations:TO-220, symbol LM7824CT
- removed U2: LM7805CT, Power_Integrations:TO-220, symbol LM7805CT
- added 4A1: Fuse, Fuse_Holders_and_Fuses:Fuse_SMD1206_Reflow, symbol F_Small
- added C16: 10uF, Capacitors_SMD:C_0603, symbol C
- added C17: 47uF, Capacitors_SMD:C_0603, symbol CP
- added C?: 0.01uF, Capacitors_SMD:C_0603, symbol C
- added D2: D_Schottky, Diodes_SMD:SOD-523, symbol D_Schottky
- added D3: TVS, Diodes_SMD:SOD-523, symbol TVS
- added D4: B340A-13-F, Diodes_SMD:SOD-523, symbol D_Schottky
- added L1: 68uH, Inductors:SELF-WE-TPC_M, symbol INDUCTOR_SMALL
- added P3, P5, P6: CONN_01X04, plc:Terminalbloc_1726040, symbol CONN_01X04
- added P7: CONN_02X06, Pin_Headers:Pin_Header_Straight_2x06, symbol CONN_02X06
- added R100: 10K, Resistors_SMD:R_0603, symbol R
- added R101: 3.24K, Resistors_SMD:R_0603, symbol R
- added R102, R103: R, Resistors_SMD:R_0603, symbol R
- added U1: TPS5420D, Housings_SOIC:SOIC-8_3.9x4.9mm_Pitch1.27mm, symbol TPS5430DDA
- C3, C4: value 0.33uF -> 0.1uF
- C5, C6: value 0.1uF -> 10uF
Connections:
- net labels added: GNDREF, I_1, I_10, I_11, I_12, I_13, I_14, I_15, I_16, I_2, I_3, I_4, I_5, I_6, I_7, I_8, I_9, PA0, PA2, PA3, PA4, PA5, PA6, PA7, PA8, PD2
- net labels removed: RS485_CTS, RS485_RX, RS485_TX
- wire segments 197 -> 281
- no-connect marks 1 -> 5
Other:
- moved on the sheet: C10, C11, C12, C13, C14, C15, C7, C8, C9, CON1, CON2, R1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

Commit message: Update schematics after Benoit's review.
Parts:
- removed C10, C7: 10uF, Capacitors_SMD:C_0603, symbol C
- removed D2: D_Schottky, Diodes_SMD:SOD-523, symbol D_Schottky
- removed P1: SERIAL_DBG, Pin_Headers:Pin_Header_Straight_1x04, symbol CONN_01X04
- removed U3: LD1117S33TR, TO_SOT_Packages_SMD:SOT-223, symbol LD1117S33TR
- removed U5: MCP2551-I/SN, Housings_SOIC:SOIC-8_3.9x4.9mm_Pitch1.27mm, symbol MCP2551-I/SN
- added D2: D_Small, symbol D_Small
- added L2: INDUCTOR_SMALL, symbol INDUCTOR_SMALL
- added P1: CONN_01X06, symbol CONN_01X06
- added U2: ISO1050, symbol ISO1050
- C1, C2: value 20pF -> 18pF
- C13, C14, C15: value 100nF -> 100pF
- C4: value 0.1uF -> 100pF
- C5, C6: value 10uF -> C; footprint Capacitors_SMD:C_0603 -> (none)
- F1: renamed from 4A1; value Fuse -> 4A
- R1: value 1k -> 10k; footprint Resistors_SMD:R_0603 -> (none)
- R101: value 3.24K -> 5.873K
- Y1: footprint Crystals_Oscillators_SMD:crystal_FA238-TSX3225 -> Crystals:Crystal_FOX-FE_SMD
- gave numbers to parts that had none: 1
Connections:
- net labels removed: +5V
- wire segments 281 -> 270
- no-connect marks 5 -> 7
Other:
- moved on the sheet: C16, C3, C4, R99

Commit message: Reprise du schéma
Refonte du schéma :
-Mise en place d'un schéma hiérarchique
-Création des pages CAN, Inputs, Outputs, Alimentation.
Parts:
- removed C1, C2: 18pF, Capacitors_SMD:C_0603, symbol C
- removed C11, C12, C8, C9: 100nF, Capacitors_SMD:C_0603, symbol C
- removed C13, C14, C15, C4: 100pF, Capacitors_SMD:C_0603, symbol C
- removed C16: 10uF, Capacitors_SMD:C_0603, symbol C
- removed C17: 47uF, Capacitors_SMD:C_0603, symbol CP
- removed C18: 0.01uF, Capacitors_SMD:C_0603, symbol C
- removed C3: 0.1uF, Capacitors_SMD:C_0603, symbol C
- removed C5, C6: C, symbol C
- removed CON1, CON2: TerminalBlock, plc:Terminalblock_1708084, symbol TerminalBlock
- removed D1: LED, LEDs:LED-0603, symbol LED
- removed D2: D_Small, symbol D_Small
- removed D3: TVS, Diodes_SMD:SOD-523, symbol TVS
- removed D4: B340A-13-F, Diodes_SMD:SOD-523, symbol D_Schottky
- removed F1: 4A, Fuse_Holders_and_Fuses:Fuse_SMD1206_Reflow, symbol F_Small
- removed JP1: Jumper_NO_Small, Wire_Pads:SolderWirePad_2x_0-8mmDrill, symbol Jumper_NO_Small
- removed L1: 68uH, Inductors:SELF-WE-TPC_M, symbol INDUCTOR_SMALL
- removed L2: INDUCTOR_SMALL, symbol INDUCTOR_SMALL
- removed P1: CONN_01X06, symbol CONN_01X06
- removed P2: CONN_01X06, Pin_Headers:Pin_Header_Straight_1x06, symbol CONN_01X06
- removed P3, P4, P5, P6: CONN_01X04, plc:Terminalbloc_1726040, symbol CONN_01X04
- removed P7: CONN_02X06, Pin_Headers:Pin_Header_Straight_2x06, symbol CONN_02X06
- removed R1: 10k, symbol R
- removed R100: 10K, Resistors_SMD:R_0603, symbol R
- removed R101: 5.873K, Resistors_SMD:R_0603, symbol R
- removed R102, R103: R, Resistors_SMD:R_0603, symbol R
- removed R2: 510, Resistors_SMD:R_0603, symbol R
- removed R99: 120, Resistors_SMD:R_0603, symbol R
- removed U1: TPS5420D, Housings_SOIC:SOIC-8_3.9x4.9mm_Pitch1.27mm, symbol TPS5430DDA
- removed U2: ISO1050, symbol ISO1050
- removed U4: STM32F105R8, Housings_QFP:LQFP-64_10x10mm_Pitch0.5mm, symbol STM32F105R8
- removed Y1: 8MHz, Crystals:Crystal_FOX-FE_SMD, symbol Crystal
Connections:
- net labels removed: +3V3, CANH, CANL, CAN_RX, CAN_TX, DBG_RX, DBG_TX, GNDREF, I_1, I_10, I_11, I_12, I_13, I_14, I_15, I_16, I_2, I_3, I_4, I_5, I_6, I_7, I_8, I_9, NRST, O_0, O_1, O_10, O_11, O_12, O_13, O_14, O_15, O_2, O_3, O_4, O_5, O_6, O_7, O_8, O_9, PA0, PA2, PA3, PA4, PA5, PA6, PA7, PA8, PD2, SWCLK, SWDIO, VIN
- wire segments 270 -> 54
- no-connect marks 7 -> 0
Other:
- note removed: "Indicator LED"
