File: hw/calaos_plc_io/calaos_plc_io_inputs-1.sch (KiCad schematic (older format))
At the start: 7 parts, among them U7 PCA9505, U8 LTV-847

Commit message: Update schematics
Parts:
- added D1, D10, D11, D12, D13, D14, D15, D16, D17, D18, D19, D2, D20, D3, D4, D5, D6, D7, D8, D9: LED, LEDs:LED-0603, symbol LED
- added D101, D22, D23, D24, D27, D28, D29, D30, D31, D32, D33, D34, D35, D36, D37, D38, D39, D40, D41: TVS 3v3, Diodes_SMD:SOD-523, symbol TVS
- added Q1: Q_NPN_BCE, Housings_SOT-23_SOT-143_TSOT-6:SOT-23, symbol Q_NPN_BCE
- added Q10, Q11, Q12, Q13, Q14, Q15, Q16, Q17, Q18, Q19, Q2, Q20, Q3, Q4, Q5, Q6, Q7, Q8, Q9: Q_NPN_BCE, Housings_SOT-23_SOT-143_TSOT-6:SOT-23_Handsoldering, symbol Q_NPN_BCE
- added R10, R11, R12, R13, R14, R15, R16, R33, R34, R35, R36, R37, R38, R39, R40, R57, R58, R67, R68, R9: 220, Resistors_SMD:R_0603, symbol R
- added R100, R101, R102, R103, R104, R105, R111, R112, R113, R114, R115, R116, R117, R118, R119, R120, R63, R64, R65, R66, R69, R70, R71, R72, R81, R82, R83, R84, R85, R86, R87, R88, R89, R90, R96, R97, R98, R99: 390, Resistors_SMD:R_0603, symbol R
- added R106, R107, R108, R109, R110, R121, R122, R123, R124, R125, R17, R18, R19, R20, R21, R22, R23, R24, R25, R26, R27, R28, R29, R30, R31, R32, R41, R42, R43, R44, R45, R46, R47, R48, R49, R50, R51, R52, R53, R54, R55, R56, R59, R60, R61, R62, R73, R74, R75, R76, R77, R78, R79, R80, R91, R92, R93, R94, R95: 10k, Resistors_SMD:R_0603, symbol R
- added U10, U11, U12, U3, U9: LTV-847, Housings_SOIC:SOIC-16_3.9x9.9mm_Pitch1.27mm, symbol TLP291-4
- added U13, U14, U15, U16: LTV-847, Housings_SOIC:SOIC-16_3.9x9.9mm_Pitch1.27mm, symbol OPTO-TRANSISTOR-4
- added unit 2 of U8
- added unit 3 of U8
- added unit 4 of U8
- D21: renamed from D2; footprint (none) -> Diodes_SMD:SOD-523
- R5, R6, R7, R8: footprint (none) -> Resistors_SMD:R_0603
- U7: footprint (none) -> Housings_SSOP:TSSOP-56_6.1x14mm_Pitch0.5mm
- U8: footprint (none) -> Housings_SOIC:SOIC-16_3.9x9.9mm_Pitch1.27mm
Connections:
- net labels added: +24V, DI_02, DI_03, DI_04, DI_05, DI_06, DI_07, DI_08, DI_09, DI_10, DI_11, DI_12, DI_13, DI_14, DI_15, DI_16, DI_17, DI_18, DI_19, DI_20, DO_01, DO_02, DO_03, DO_04, DO_05, DO_06, DO_07, DO_08, DO_09, DO_10, DO_11, DO_12, DO_13, DO_14, DO_15, DO_16, DO_17, DO_18, DO_19, DO_20, INT, I_0, I_1, I_10, I_11, I_12, I_13, I_14, I_15, I_16, I_17, I_18, I_19, I_2, I_3, I_4, I_5, I_6, I_7, I_8, I_9, O_0, O_1, O_10, O_11, O_12, O_13, O_14, O_15, O_16, O_17, O_18, O_19, O_2, O_3, O_4, O_5, O_6, O_7, O_8, O_9
- net labels removed: I0_0, I0_1, I0_2, I0_3, I0_4, I0_5, I0_6, I0_7, I1_0, I1_1, I1_2, I1_3, I1_4, I1_5, I1_6, I1_7, I2_0, I2_1, I2_2, I2_3, I2_4, I2_5, I2_6, I2_7, I3_0, I3_1, I3_2, I3_3, I3_4, I3_5, I3_6, I3_7, I4_0, I4_1, I4_2, I4_3, I4_4, I4_5, I4_6, I4_7, INT_INPUTS
- wire segments 72 -> 659
Other:
- moved on the sheet: R5, R6, R7, R8

Commit message: Add pcb with placement of components
Parts:
- removed D1, D10, D11, D12, D13, D14, D15, D16, D17, D18, D19, D2, D20, D3, D4, D5, D6, D7, D8, D9: LED, LEDs:LED-0603, symbol LED
- removed D38, D39, D40, D41: TVS 3v3, Diodes_SMD:SOD-523, symbol TVS
- removed Q17, Q18, Q19, Q20: Q_NPN_BCE, Housings_SOT-23_SOT-143_TSOT-6:SOT-23_Handsoldering, symbol Q_NPN_BCE
- removed R112, R113, R114, R115, R117, R118, R119, R120: 390, Resistors_SMD:R_0603, symbol R
- removed R122, R123, R124, R125, R59, R60, R61, R62, R73, R74, R79, R8, R80: 10k, Resistors_SMD:R_0603, symbol R
- removed R57, R58, R67, R68: 220, Resistors_SMD:R_0603, symbol R
- removed U12: LTV-847, Housings_SOIC:SOIC-16_3.9x9.9mm_Pitch1.27mm, symbol TLP291-4
- removed U16: LTV-847, Housings_SOIC:SOIC-16_3.9x9.9mm_Pitch1.27mm, symbol OPTO-TRANSISTOR-4
- removed U7: PCA9505, Housings_SSOP:TSSOP-56_6.1x14mm_Pitch0.5mm, symbol PCA9505
- Q10, Q11, Q12, Q13, Q14, Q15, Q16, Q2, Q3, Q4, Q5, Q6, Q7, Q8, Q9: footprint Housings_SOT-23_SOT-143_TSOT-6:SOT-23_Handsoldering -> Housings_SOT-23_SOT-143_TSOT-6:SOT-23
- renumbered D21 to D18, D101 to D19, D22 to D20, D23 to D21, D24 to D22, D27 to D23, D28 to D24, D29 to D25, D30 to D26, D31 to D27, D32 to D28, D33 to D29, D34 to D30, D35 to D31, D36 to D32, D37 to D33, R16 to R10, R17 to R11, R18 to R12, R19 to R13, R20 to R14, R21 to R15, R22 to R16, R23 to R17, R24 to R18, R25 to R19, R26 to R20, R27 to R21, R28 to R22, R29 to R23, R30 to R24, R31 to R25, R32 to R26, R33 to R27, R34 to R28, R35 to R29, R9 to R3, R36 to R30, R37 to R31, R38 to R32, R39 to R33, R40 to R34, R41 to R35, R42 to R36, R43 to R37, R44 to R38, R45 to R39, R10 to R4, R46 to R40, R47 to R41, R48 to R42, R49 to R43, R50 to R44, R51 to R45, R52 to R46, R53 to R47, R54 to R48, R55 to R49, R11 to R5, R56 to R50, R5 to R51, R63 to R52, R64 to R53, R65 to R54, R66 to R55, R6 to R56, R69 to R57, R70 to R58, R71 to R59, R12 to R6, R72 to R60, R7 to R61, R75 to R62, R76 to R63, R77 to R64, R78 to R65, R81 to R66, R82 to R67, R83 to R68, R84 to R69, R13 to R7, R85 to R70, R86 to R71, R87 to R72, R88 to R73, R89 to R74, R90 to R75, R91 to R76, R92 to R77, R93 to R78, R94 to R79, R14 to R8, R95 to R80, R96 to R81, R97 to R82, R98 to R83, R99 to R84, R100 to R85, R101 to R86, R102 to R87, R103 to R88, R104 to R89, R15 to R9, R105 to R90, R106 to R91, R107 to R92, R108 to R93, R109 to R94, R110 to R95, R111 to R96, R116 to R97, R121 to R98, U8 to U10, U13 to U11, U14 to U12, U15 to U13, U3 to U6, U9 to U7, U10 to U8, U11 to U9
Connections:
- net labels removed: DI_17, DI_18, DI_19, DI_20, DO_17, DO_18, DO_19, DO_20, INT, I_16, I_17, I_18, I_19, O_16, O_17, O_18, O_19, SCL, SDA
- wire segments 659 -> 464
Other:
- note removed: "I2C address : 0x40"

Commit message: Update schematics and pcb
Connections:
- net labels added: +24v, +5v, I_16
- net labels removed: I_0
- wire segments 464 -> 472
Other:
- moved on the sheet: R10, R11, R12, R13, R14, R15, R16, R17, R18, R19, R20, R21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

Commit message: Update schematics after Benoit's review.
Parts:
- removed D18, D19, D20, D21, D22, D23, D24, D25, D26, D27, D28, D29, D30, D31, D32, D33: TVS 3v3, Diodes_SMD:SOD-523, symbol TVS
- removed Q1, Q10, Q11, Q12, Q13, Q14, Q15, Q16, Q2, Q3, Q4, Q5, Q6, Q7, Q8, Q9: Q_NPN_BCE, Housings_SOT-23_SOT-143_TSOT-6:SOT-23, symbol Q_NPN_BCE
- added D10, D11, D12, D13, D14, D15, D16, D17, D18, D19, D20, D5, D6, D7, D8, D9: D, symbol D
- added Q? (x16): Q_NMOS_GDS, symbol Q_NMOS_GDS
Connections:
- net labels added: +3V3, +3v3
- net labels removed: +5V, +5v
- wire segments 472 -> 488
Other:
- note removed: "30mA @ 24V\n25mA @ 12V\n5mA @ 5V\n=> 35V -> 5V input \nwith opto like LTV-847 ?"

Commit message: Reprise du schéma
Refonte du schéma :
-Mise en place d'un schéma hiérarchique
-Création des pages CAN, Inputs, Outputs, Alimentation.
Parts:
- removed D10, D11, D12, D13, D14, D15, D16, D17, D18, D19, D20, D5, D6, D7, D8, D9: D, symbol D
- removed Q? (x16): Q_NMOS_GDS, symbol Q_NMOS_GDS
- removed R10, R27, R28, R29, R3, R30, R31, R32, R33, R34, R4, R5, R6, R7, R8, R9: 220, Resistors_SMD:R_0603, symbol R
- removed R11, R12, R13, R14, R15, R16, R17, R18, R19, R20, R21, R22, R23, R24, R25, R26, R35, R36, R37, R38, R39, R40, R41, R42, R43, R44, R45, R46, R47, R48, R49, R50, R61, R62, R63, R64, R65, R76, R77, R78, R79, R80, R91, R92, R93, R94, R95, R98: 10k, Resistors_SMD:R_0603, symbol R
- removed R51, R52, R53, R54, R55, R56, R57, R58, R59, R60, R66, R67, R68, R69, R70, R71, R72, R73, R74, R75, R81, R82, R83, R84, R85, R86, R87, R88, R89, R90, R96, R97: 390, Resistors_SMD:R_0603, symbol R
- removed U10, U11, U12, U13: LTV-847, Housings_SOIC:SOIC-16_3.9x9.9mm_Pitch1.27mm, symbol OPTO-TRANSISTOR-4
- removed U6, U7, U8, U9: LTV-847, Housings_SOIC:SOIC-16_3.9x9.9mm_Pitch1.27mm, symbol TLP291-4
- added CON501, CON502, CON503, CON504: TerminalBlock, plc:Terminalblock_1708084, symbol TerminalBlock
Connections:
- net labels added: +3.3V, O_16
- net labels removed: +3V3, DI_01, DI_02, DI_03, DI_04, DI_05, DI_06, DI_07, DI_08, DI_09, DI_10, DI_11, DI_12, DI_13, DI_14, DI_15, DI_16, DO_01, DO_02, DO_03, DO_04, DO_05, DO_06, DO_07, DO_08, DO_09, DO_10, DO_11, DO_12, DO_13, DO_14, DO_15, DO_16, GNDREF, O_0
- wire segments 488 -> 110
