File: hw/nucleo_shield/nucleo_shield_output.sch (KiCad schematic (older format))
At the start: 10 parts, among them P10 CONN_OUTH1, P11 CONN_OUTH2, P2 CONN_OUT3, P8 CONN_OUT4, U1 74HC595, U10 ULN2803, U11 74HC595, U12 74HC595, U2 74HC595, U9 ULN2803

Commit message: HW: rework of nucleo shield to add more IOs
Parts:
- P2, P8: footprint Pin_Headers:Pin_Header_Straight_1x08 -> Pin_Headers:Pin_Header_Straight_1x10; symbol CONN_01X08 -> CONN_01X10
Connections:
- net SRCLK2 is gone; now on net SRCLK: U11.11 (SRCLK), U12.11 (SRCLK)
- net SRDATA2 is gone; now on an unnamed net: U11.14 (SER)
- net SRLatch2 is gone; now on net SRLatch: U11.12 (RCLK), U12.12 (RCLK)
- net +5V: now also P2.2 (P2), P8.9 (P9)
- net GND: now also P2.1 (P1), P8.10 (P10)
- net SRCLK: now also U2.11 (SRCLK)
- net SRLatch: now also U2.12 (RCLK)
- net out17: now also P2.10 (P10); no longer P2.8 (P8)
- net out18: now also P2.9 (P9); no longer P2.7 (P7)
- net out19: now also P2.8 (P8); no longer P2.6 (P6)
- net out20: now also P2.7 (P7); no longer P2.5 (P5)
- net out21: now also P2.6 (P6); no longer P2.4 (P4)
- net out22: now also P2.5 (P5); no longer P2.3 (P3)
- net out23: now also P2.4 (P4); no longer P2.2 (P2)
- net out24: now also P2.3 (P3); no longer P2.1 (P1)
Changed lines of the file:
@@
 $Descr A4 11693 8268
 encoding utf-8
-Sheet 2 4
+Sheet 4 4
 Title ""
 Date ""
@@
 $EndComp
 $Comp
-L GND #PWR030
+L GND #PWR052
 U 1 1 5729AB4A
 P 1500 1900
-F 0 "#PWR030" H 1500 1650 50  0001 C CNN
+F 0 "#PWR052" H 1500 1650 50  0001 C CNN
 F 1 "GND" H 1500 1750 50  0000 C CNN
 F 2 "" H 1500 1900 60  0000 C CNN
@@
 $EndComp
 $Comp
-L GND #PWR031
+L GND #PWR053
 U 1 1 5729AB50
 P 1500 3500
-F 0 "#PWR031" H 1500 3250 50  0001 C CNN
+F 0 "#PWR053" H 1500 3250 50  0001 C CNN
 F 1 "GND" H 1500 3350 50  0000 C CNN
 F 2 "" H 1500 3500 60  0000 C CNN
@@
 $EndComp
 $Comp
-L +5V #PWR032
+L +5V #PWR054
 U 1 1 5729ABD5
 P 1900 750
-F 0 "#PWR032" H 1900 600 50  0001 C CNN
+F 0 "#PWR054" H 1900 600 50  0001 C CNN
 F 1 "+5V" H 1900 890 50  0000 C CNN
 F 2 "" H 1900 750 60  0000 C CNN
@@
 $EndComp
 $Comp
-L +5V #PWR033
+L +5V #PWR055
 U 1 1 5729ABDB
 P 3600 2400
-F 0 "#PWR033" H 3600 2250 50  0001 C CNN
+F 0 "#PWR055" H 3600 2250 50  0001 C CNN
 F 1 "+5V" H 3600 2540 50  0000 C CNN
 F 2 "" H 3600 2400 60  0000 C CNN
@@
 $EndComp
 $Comp
-L +5V #PWR034
+L +5V #PWR056
 U 1 1 5729ABE8
 P 1350 1450
-F 0 "#PWR034" H 1350 1300 50  0001 C CNN
+F 0 "#PWR056" H 1350 1300 50  0001 C CNN
 F 1 "+5V" H 1350 1590 50  0000 C CNN
 F 2 "" H 1350 1450 60  0000 C CNN
@@
 $EndComp
 $Comp
-L +5V #PWR035
+L +5V #PWR057
 U 1 1 5729ABEE
 P 1100 2950
-F 0 "#PWR035" H 1100 2800 50  0001 C CNN
+F 0 "#PWR057" H 1100 2800 50  0001 C CNN
 F 1 "+5V" H 1100 3090 50  0000 C CNN
 F 2 "" H 1100 2950 60  0000 C CNN
@@
 $EndComp
 $Comp
-L GND #PWR036
+L GND #PWR058
 U 1 1 57307D6B
 P 7150 1750
-F 0 "#PWR036" H 7150 1500 50  0001 C CNN
+F 0 "#PWR058" H 7150 1500 50  0001 C CNN
 F 1 "GND" H 7150 1600 50  0000 C CNN
 F 2 "" H 7150 1750 60  0000 C CNN
@@
 $EndComp
 $Comp
-L GND #PWR037
+L GND #PWR059
 U 1 1 57307D82
 P 7600 3400
-F 0 "#PWR037" H 7600 3150 50  0001 C CNN
+F 0 "#PWR059" H 7600 3150 50  0001 C CNN
 F 1 "GND" H 7600 3250 50  0000 C CNN
 F 2 "" H 7600 3400 60  0000 C CNN
@@
 $EndComp
 $Comp
-L +24V #PWR038
+L +24V #PWR060
 U 1 1 57307DA1
 P 7150 750
-F 0 "#PWR038" H 7150 600 50  0001 C CNN
+F 0 "#PWR060" H 7150 600 50  0001 C CNN
 F 1 "+24V" H 7150 890 50  0000 C CNN
 F 2 "" H 7150 750 60  0000 C CNN
@@
 out8h
 $Comp
-L CONN_01X08 P2
+L CONN_01X10 P2
 U 1 1 57326C94
-P 5500 4750
-F 0 "P2" H 5500 5300 50  0000 C CNN
-F 1 "CONN_OUT3" V 5600 4750 50  0000 C CNN
-F 2 "Pin_Headers:Pin_Header_Straight_1x08" H 5500 4750 60  0001 C CNN
-F 3 "" H 5500 4750 60  0000 C CNN
-	1    5500 4750
+P 5500 4650
+F 0 "P2" H 5500 5200 50  0000 C CNN
+F 1 "CONN_OUT3" V 5600 4650 50  0000 C CNN
+F 2 "Pin_Headers:Pin_Header_Straight_1x10" H 5500 4650 60  0001 C CNN
+F 3 "" H 5500 4650 60  0000 C CNN
+	1    5500 4650
 	1    0    0    -1
 $EndComp
@@
 out18
 $Comp
-L +5V #PWR039
+L +5V #PWR061
 U 1 1 57326A4A
 P 950 4650
-F 0 "#PWR039" H 950 4500 50  0001 C CNN
+F 0 "#PWR061" H 950 4500 50  0001 C CNN
 F 1 "+5V" H 950 4790 50  0000 C CNN
 F 2 "" H 950 4650 60  0000 C CNN
@@
 $EndComp
 $Comp
-L GND #PWR040
+L GND #PWR062
 U 1 1 57326A1D
 P 1500 5100
-F 0 "#PWR040" H 1500 4850 50  0001 C CNN
+F 0 "#PWR062" H 1500 4850 50  0001 C CNN
 F 1 "GND" H 1500 4950 50  0000 C CNN
 F 2 "" H 1500 5100 60  0000 C CNN
@@
 $EndComp
 $Comp
-L +5V #PWR041
+L +5V #PWR063
 U 1 1 5733141E
 P 3600 5600
-F 0 "#PWR041" H 3600 5450 50  0001 C CNN
+F 0 "#PWR063" H 3600 5450 50  0001 C CNN
 F 1 "+5V" H 3600 5740 50  0000 C CNN
 F 2 "" H 3600 5600 60  0000 C CNN
@@
 out26
 $Comp
-L +5V #PWR042
+L +5V #PWR064
 U 1 1 5733142A
 P 1100 6150
-F 0 "#PWR042" H 1100 6000 50  0001 C CNN
+F 0 "#PWR064" H 1100 6000 50  0001 C CNN
 F 1 "+5V" H 1100 6290 50  0000 C CNN
 F 2 "" H 1100 6150 60  0000 C CNN
@@
 $EndComp
 $Comp
-L GND #PWR043
+L GND #PWR065
 U 1 1 57331432
 P 1500 6700
-F 0 "#PWR043" H 1500 6450 50  0001 C CNN
+F 0 "#PWR065" H 1500 6450 50  0001 C CNN
 F 1 "GND" H 1500 6550 50  0000 C CNN
 F 2 "" H 1500 6700 60  0000 C CNN
@@
 $EndComp
 $Comp
-L CONN_01X08 P8
+L CONN_01X10 P8
 U 1 1 57331532
-P 5900 6250
-F 0 "P8" H 5900 6800 50  0000 C CNN
-F 1 "CONN_OUT4" V 6000 6250 50  0000 C CNN
-F 2 "Pin_Headers:Pin_Header_Straight_1x08" H 5900 6250 60  0001 C CNN
-F 3 "" H 5900 6250 60  0000 C CNN
-	1    5900 6250
+P 5900 6350
+F 0 "P8" H 5900 6900 50  0000 C CNN
+F 1 "CONN_OUT4" V 6000 6350 50  0000 C CNN
+F 2 "Pin_Headers:Pin_Header_Straight_1x10" H 5900 6350 60  0001 C CNN
+F 3 "" H 5900 6350 60  0000 C CNN
+	1    5900 6350
 	1    0    0    -1
 $EndComp
@@
 out31
 $Comp
-L +24V #PWR044
+L +24V #PWR066
 U 1 1 57334377
 P 7600 2100
-F 0 "#PWR044" H 7600 1950 50  0001 C CNN
+F 0 "#PWR066" H 7600 1950 50  0001 C CNN
 F 1 "+24V" H 7600 2240 50  0000 C CNN
 F 2 "" H 7600 2100 60  0000 C CNN
@@
 	1    0    0    -1
 $EndComp
-Text HLabel 950  4250 0    60   Input ~ 0
-SRDATA2
-Text HLabel 850  4450 0    60   Input ~ 0
-SRCLK2
-Text HLabel 900  4750 0    60   Input ~ 0
-SRLatch2
-$Comp
-L +5V #PWR045
+$Comp
+L +5V #PWR067
 U 1 1 576808E1
-P 2150 4000
-F 0 "#PWR045" H 2150 3850 50  0001 C CNN
-F 1 "+5V" H 2150 4140 50  0000 C CNN
-F 2 "" H 2150 4000 60  0000 C CNN
-F 3 "" H 2150 4000 60  0000 C CNN
-	1    2150 4000
-	1    0    0    -1
-$EndComp
-Wire Wire Line
-	2150 4050 2150 4000
-Wire Wire Line
-	1900 4050 2150 4050
+P 3300 4050
+F 0 "#PWR067" H 3300 3900 50  0001 C CNN
+F 1 "+5V" H 3300 4190 50  0000 C CNN
+F 2 "" H 3300 4050 60  0000 C CNN
+F 3 "" H 3300 4050 60  0000 C CNN
+	1    3300 4050
+	1    0    0    -1
+$EndComp
+Wire Wire Line
+	1900 4050 3300 4050
 Wire Wire Line
 	1900 4150 1900 4050
 Wire Wire Line
-	950  4250 1500 4250
-Wire Wire Line
 	950  4650 1500 4650
 Wire Wire Line
-	1200 6050 1200 4450
-Wire Wire Line
-	1050 4750 1050 6350
+	1200 1250 1200 6050
+Wire Wire Line
+	1050 1550 1050 6350
 Wire Wire Line
 	7600 2400 7600 2100
@@
 Wire Wire Line
 	5700 6600 5400 6600
-Connection ~ 1200 4450
-Connection ~ 1050 4750
 Wire Wire Line
 	1500 5850 1500 5400
@@
 Wire Wire Line
 	2900 2650 3200 2650
-Wire Wire Line
-	850  4450 1500 4450
-Wire Wire Line
-	900  4750 1500 4750
 Wire Wire Line
 	1500 4850 1500 5100
@@
 Wire Wire Line
 	1500 1650 1500 1900
+$Comp
+L +5V #PWR068
+U 1 1 5769D296
+P 5050 7000
+F 0 "#PWR068" H 5050 6850 50  0001 C CNN
+F 1 "+5V" H 5050 7140 50  0000 C CNN
+F 2 "" H 5050 7000 60  0000 C CNN
+F 3 "" H 5050 7000 60  0000 C CNN
+	1    5050 7000
+	-1   0    0    1
+$EndComp
+$Comp
+L GND #PWR069
+U 1 1 5769D305
+P 5600 7000
+F 0 "#PWR069" H 5600 6750 50  0001 C CNN
+F 1 "GND" H 5600 6850 50  0000 C CNN
+F 2 "" H 5600 7000 60  0000 C CNN
+F 3 "" H 5600 7000 60  0000 C CNN
+	1    5600 7000
+	1    0    0    -1
+$EndComp
+Wire Wire Line
+	5700 6700 5050 6700
+Wire Wire Line
+	5050 6700 5050 7000
+Wire Wire Line
+	5600 7000 5600 6800
+Wire Wire Line
+	5600 6800 5700 6800
+$Comp
+L +5V #PWR070
+U 1 1 5769D8BC
+P 4300 3950
+F 0 "#PWR070" H 4300 3800 50  0001 C CNN
+F 1 "+5V" H 4300 4090 50  0000 C CNN
+F 2 "" H 4300 3950 60  0000 C CNN
+F 3 "" H 4300 3950 60  0000 C CNN
+	1    4300 3950
+	1    0    0    -1
+$EndComp
+$Comp
+L GND #PWR071
+U 1 1 5769D8DB
+P 4700 3950
+F 0 "#PWR071" H 4700 3700 50  0001 C CNN
+F 1 "GND" H 4700 3800 50  0000 C CNN
+F 2 "" H 4700 3950 60  0000 C CNN
+F 3 "" H 4700 3950 60  0000 C CNN
+	1    4700 3950
+	-1   0    0    1
+$EndComp
+Wire Wire Line
+	5300 4300 4300 4300
+Wire Wire Line
+	4300 4300 4300 3950
+Wire Wire Line
+	4700 3950 4700 4200
+Wire Wire Line
+	4700 4200 5300 4200
+Wire Wire Line
+	2900 3550 2900 3950
+Wire Wire Line
+	2900 3950 1500 3950
+Wire Wire Line
+	1500 3950 1500 4250
+Wire Wire Line
+	1500 4450 1200 4450
+Connection ~ 1200 4450
+Wire Wire Line
+	1500 4750 1050 4750
+Connection ~ 1050 4750
 $EndSCHEMATC
