File: hw/nucleo_shield/nucleo_shield_input.sch (KiCad schematic (older format))
At the start: 38 parts, among them P1 CONN_INH1, P5 CONN_INH2, U3 LTV-847, U4 LTV-847, U5 LTV-847, U6 LTV-847

Commit message: WIP: add more IO
Parts:
- added P17: CONN_INH3, w_conn_screw:mors_8p, symbol CONN_01X08
- added R34, R37, R38, R39, R40, R41, R42, R43: R, Resistors_ThroughHole:Resistor_Horizontal_RM10mm, symbol R
- added R44, R45, R46, R47, R48, R49, R50, R51: R, Resistors_SMD:R_0805_HandSoldering, symbol R
- added U15, U16: LTV-847, Housings_DIP:DIP-16__300, symbol LTV-847
- P1, P5: footprint w_conn_screw:mors_10p -> w_conn_screw:mors_8p; symbol CONN_01X10 -> CONN_01X08
Connections:
- net +3V3: now also U15.10, U15.12, U15.14, U15.16, U16.10, U16.12, U16.14, U16.16
- net GND: now also R44.1, R45.1, R46.1, R47.1, R48.1, R49.1, R50.1, R51.1
- net GND_24V: now also U15.2, U15.4, U15.6, U15.8, U16.2, U16.4, U16.6, U16.8; no longer P1.1 (P1), P1.2 (P2), P5.1 (P1), P5.2 (P2)
- net inh1: now also P1.5 (P5); no longer P1.7 (P7)
- net inh10: now also P5.7 (P7); no longer P5.9 (P9)
- net inh11: now also P5.5 (P5); no longer P5.7 (P7)
- net inh12: now also P5.6 (P6); no longer P5.8 (P8)
- net inh13: now also P5.4 (P4); no longer P5.6 (P6)
- net inh14: now also P5.3 (P3); no longer P5.5 (P5)
- net inh15: now also P5.2 (P2); no longer P5.4 (P4)
- net inh16: now also P5.1 (P1); no longer P5.3 (P3)
- net inh2: now also P1.6 (P6); no longer P1.8 (P8)
- net inh3: now also P1.7 (P7); no longer P1.9 (P9)
- net inh4: now also P1.8 (P8); no longer P1.10 (P10)
- net inh5: now also P1.1 (P1); no longer P1.3 (P3)
- net inh6: now also P1.2 (P2); no longer P1.4 (P4)
- net inh7: now also P1.3 (P3); no longer P1.5 (P5)
- net inh8: now also P1.4 (P4); no longer P1.6 (P6)
- net inh9: now also P5.8 (P8); no longer P5.10 (P10)
- new net: R40.1, U16.1
- new net: R41.1, U16.3
- new net: R42.1, U16.5
- new net: R43.1, U16.7
- new net: R34.1, U15.1
- new net: R37.1, U15.3
- new net: R38.1, U15.5
- new net: R39.1, U15.7
- new net in17: R51.2, U16.15
- new net in18: R49.2, U16.13
- new net in19: R47.2, U16.11
- new net in20: R45.2, U16.9
- new net in21: R50.2, U15.15
- new net in22: R48.2, U15.13
- new net in23: R46.2, U15.11
- new net in24: R44.2, U15.9
- new net inh17: P17.8 (P8), R40.2
- new net inh18: P17.7 (P7), R41.2
- new net inh19: P17.6 (P6), R42.2
- new net inh20: P17.5 (P5), R43.2
- new net inh21: P17.4 (P4), R34.2
- new net inh22: P17.3 (P3), R37.2
- new net inh23: P17.2 (P2), R38.2
- new net inh24: P17.1 (P1), R39.2
Other:
- moved on the sheet: R1, R10, R11, R12, R13, R14, R15, R16, R17, R18, R19, R2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

Commit message: HW: rework of nucleo shield to add more IOs
Parts:
- R1, R17, R18, R19, R2, R20, R25, R26, R27, R28, R3, R34, R37, R38, R39, R4, R40, R41, R42, R43, R5, R6, R7, R8: footprint Resistors_ThroughHole:Resistor_Horizontal_RM10mm -> Resistors_SMD:R_0805_HandSoldering
Connections:
- net in17: now also R44.2, U15.9; no longer R51.2, U16.15
- net in18: now also R46.2, U15.11; no longer R49.2, U16.13
- net in19: now also R48.2, U15.13; no longer R47.2, U16.11
- net in20: now also R50.2, U15.15; no longer R45.2, U16.9
- net in21: now also R51.2, U16.15; no longer R50.2, U15.15
- net in22: now also R49.2, U16.13; no longer R48.2, U15.13
- net in23: now also R47.2, U16.11; no longer R46.2, U15.11
- net in24: now also R45.2, U16.9; no longer R44.2, U15.9
- net inh17: now also R43.2; no longer R40.2
- net inh18: now also R42.2; no longer R41.2
- net inh19: now also R41.2; no longer R42.2
- net inh20: now also R40.2; no longer R43.2
- net inh21: now also R39.2; no longer R34.2
- net inh22: now also R38.2; no longer R37.2
- net inh23: now also R37.2; no longer R38.2
- net inh24: now also R34.2; no longer R39.2
